File: Power.kicad_sch (KiCad schematic)
At the start: 43 parts, among them U2 LMR33630CRNXR, U3 LMR33630CRNXR, U4 NCP187AMT330TAG, U5 TCR3RM33A

Commit message: Crystal change, gnd cut-out for crystal, bom update
Parts:
- C16, C17, C18, C20: Unit Price 0.3533 -> (none)
- C19, C21, C23, C24: Unit Price 0.0401 -> (none)
- C22, C25, C47, C48, C50: Unit Price 0.0060 -> (none)
- C26, C27: Unit Price 0.0030 -> (none)
- C28, C29, C31, C45: JLCPCB # C2987934 -> C86816; MANUFACTURER # GRM32ER71E226KE15L -> GRM21BR61E226ME44L; Tollerance 10% -> 20%; Unit Price 0.4635 -> (none)
- C30, C46: JLCPCB # C2987934 -> C77082; MANUFACTURER # GRM31CD71H106KE11L -> GRM21BR71H104KA01L; Unit Price 0.4635 -> (none)
- C49: Unit Price 0.0480 -> (none)
- D6, D7, D9: Ifrwd 5mA -> (none); JLCPCB # C42456066 -> C364551; MANUFACTURER Orient -> Lite-On; MANUFACTURER # ORH-G36G-B -> LTST-C281KGKT-5A; Package 0603 -> 0402; Unit Price 0.0125 -> (none)
- D8: JLCPCB # C160479 -> C364551; MANUFACTURER # LTST-C281KGKT -> LTST-C281KGKT-5A; Unit Price 0.0459 -> (none)
- L1, L2: Unit Price 0.2616 -> (none)
- R24: JLCPCB # C850952 -> C7294197; MANUFACTURER # AT0402BRD0730K1L -> RP0402BRD0724K9L; Unit Price 0.0446 -> (none)
- R28, R8: JLCPCB # C185464 -> C7294193; MANUFACTURER # RC0402FR-07158KL -> RP0402BRD07100KL; Tollerance 1% -> 0.1%; Unit Price 0.0006 -> (none)
- R29: Unit Price 0.0446 -> (none)
- R30, R31, R33, R34: Unit Price 0.0006 -> (none)
- R32: JLCPCB # C852071 -> C7294193; MANUFACTURER # RE0402FRE07100KL -> RP0402BRD07100KL; Tollerance 1% -> 0.1%; Unit Price 0.0015 -> (none)
- R35: JLCPCB # C850952 -> C7294193; MANUFACTURER # AT0402BRD0730K1L -> RP0402BRD07100KL; Unit Price 0.0446 -> (none)
- U4: Unit Price 0.8498 -> (none)
- U5: Unit Price 0.1842 -> (none)

Commit message: Updated
Parts:
- C16, C17, C18, C20: JLCPCB # C437568 -> (none); LCSC (none) -> C437568
- C19, C21, C23, C24: JLCPCB # C161262 -> (none); LCSC (none) -> C161262
- C22, C25, C47, C48, C50: JLCPCB # C77009 -> (none); LCSC (none) -> C77009
- C26, C27: JLCPCB # C77020 -> (none); LCSC (none) -> C77020
- C28, C29, C31, C45: JLCPCB # C86816 -> (none); LCSC (none) -> C86816
- C30, C46: JLCPCB # C77082 -> (none); LCSC (none) -> C77082
- C49: JLCPCB # C77093 -> (none); LCSC (none) -> C77093
- D5: LCSC (none) -> C6671609; MANUFACTURER (none) -> Diodes; MANUFACTURER # (none) -> SDM2A40CSP-7B
- D6, D7, D8, D9: JLCPCB # C364551 -> (none); LCSC (none) -> C364551
- L1, L2: JLCPCB # C494329 -> (none); LCSC (none) -> C494329
- R24: JLCPCB # C7294197 -> (none); LCSC (none) -> C7294197
- R28, R32, R35, R8: JLCPCB # C7294193 -> (none); LCSC (none) -> C7294193
- R29: JLCPCB # C850952 -> (none); LCSC (none) -> C850952
- R30, R33, R34: JLCPCB # C114877 -> (none); LCSC (none) -> C114877
- R31: JLCPCB # C114762 -> (none); LCSC (none) -> C114762
- U2, U3: LCSC (none) -> C2071783; MANUFACTURER (none) -> TI; MANUFACTURER # (none) -> LMR33630CRNXR
- U4: JLCPCB # C892299 -> (none); LCSC (none) -> C892299
- U5: JLCPCB # C5797528 -> (none); LCSC (none) -> C5797528
