File: mcu.kicad_sch (KiCad schematic)
At the start: 30 parts, among them SW1 BOOT, U1 STM32G473RET6, Y1 8MHz

Commit message: Crystal change, gnd cut-out for crystal, bom update
Parts:
- C1: JLCPCB # C2858031 -> C385032; MANUFACTURER # GRM155R61E475ME15D -> GRM155R61E225KE11D; Tollerance 20% -> 10%; Unit Price 0.0363 -> (none)
- C10: Unit Price 0.0022 -> (none)
- C11, C12, C14, C15, C2, C3, C4, C5, C9: JLCPCB # C71629 -> C77020; MANUFACTURER # GRM155R71C104KA88D -> GRM155R71H104KE14D; Unit Price 0.0016 -> (none); Voltage 16V -> 50V
- C13: Unit Price 0.0143 -> (none)
- C6: Unit Price 0.0060 -> (none)
- C7, C8: value 18p -> 24p; JLCPCB # C384967 -> C1864480; MANUFACTURER # GRM0335C1H180FA01D -> GCM1555C1H240FA16D; Unit Price 0.0068 -> (none)
- D1: Ifrwd 2mA -> (none); Unit Price 0.0410 -> (none)
- R1, R19, R20, R21, R23: Unit Price 0.0006 -> (none)
- R22: JLCPCB # C852071 -> C7294193; MANUFACTURER # RE0402FRE07100KL -> RP0402BRD07100KL; Tollerance 1% -> 0.1%; Unit Price 0.0015 -> (none)
- R9: Unit Price 0.0007 -> (none)
- SW1: Unit Price 0.1493 -> (none)
- U1: Unit Price 6.1560 -> (none)
- Y1: footprint 0_passives:Crystal_SMD_3225-4Pin_3.2x2.5mm -> 0_passives:ABM3; symbol 0_passives:Crystal_4Pin -> 0_passives:Crystal_2Pin; JLCPCB # C2595911 -> (none); MANUFACTURER ECS -> Abracon; MANUFACTURER # ECS-80-12-33Q-GN-TR -> ABM3-8.000MHZ-B4Y-T; Mouser # (none) -> 815-ABM38000B4YT; Package SMD3225-4P -> (none); Unit Price 1.2705 -> (none)
Connections:
- net GND: no longer Y1.2, Y1.4
- net MCU_OSC_OUT: now also Y1.2; no longer Y1.3

Commit message: Updated
Parts:
- C1: JLCPCB # C385032 -> (none); LCSC (none) -> C426094; MANUFACTURER # GRM155R61E225KE11D -> GRM155R61C475KE15D
- C10: JLCPCB # C77013 -> (none); LCSC (none) -> C77013
- C11, C12, C14, C15, C2, C3, C4, C5, C9: JLCPCB # C77020 -> (none); LCSC (none) -> C77020
- C13: JLCPCB # C385032 -> (none); LCSC (none) -> C385032
- C6: JLCPCB # C77009 -> (none); LCSC (none) -> C77009
- C7, C8: JLCPCB # C1864480 -> (none); LCSC (none) -> C1864480
- D1: JLCPCB # C364550 -> (none); LCSC (none) -> C364550
- R1, R19, R23: JLCPCB # C60490 -> (none); LCSC (none) -> C60490
- R20, R21: JLCPCB # C105870 -> (none); LCSC (none) -> C105870
- R22: JLCPCB # C7294193 -> (none); LCSC (none) -> C7294193
- R9: JLCPCB # C106232 -> (none); LCSC (none) -> C106232
- SW1: JLCPCB # C231329 -> (none); LCSC (none) -> C231329
- U1: JLCPCB # C730120 -> (none); LCSC (none) -> C730120
- Y1: LCSC (none) -> C5564812
