File: osd.kicad_sch (KiCad schematic)
At the start: 14 parts, among them U9 STM32G431KBU6

Commit message: Crystal change, gnd cut-out for crystal, bom update
Parts:
- C38: JLCPCB # C77013 -> C21012317; MANUFACTURER # GRM155R71E103KA01D -> GRM15XR71H561KA86J; Unit Price 0.0022 -> (none); Voltage 25V -> 50V
- C39, C41: JLCPCB # C77013 -> C77020; MANUFACTURER # GRM155R71E103KA01D -> GRM155R71H104KE14D; Unit Price 0.0022 -> (none); Voltage 25V -> 50V
- C40: Unit Price 0.0060 -> (none)
- C42, C43: JLCPCB # C71629 -> C77020; MANUFACTURER # GRM155R71C104KA88D -> GRM155R71H104KE14D; Unit Price 0.0016 -> (none); Voltage 16V -> 50V
- C44: JLCPCB # C2858031 -> C385032; MANUFACTURER # GRM155R61E475ME15D -> GRM155R61E225KE11D; Tollerance 20% -> 10%; Unit Price 0.0363 -> (none)
- FB1: JLCPCB # (none) -> C107335; MANUFACTURER (none) -> TDK; MANUFACTURER # (none) -> MPZ1608S601ATA00; Package (none) -> 0603
- R40: JLCPCB # (none) -> C137841; MANUFACTURER (none) -> YAGEO; MANUFACTURER # (none) -> RC0402JR-0775RL; Tollerance 1% -> 5%
- R41: Unit Price 0.0006 -> (none)
- R42: JLCPCB # C60490 -> C106232; MANUFACTURER # RC0402FR-0710KL -> RC0402FR-07100RL; Unit Price 0.0006 -> (none)

Commit message: Updated
Parts:
- C38: JLCPCB # C21012317 -> (none); LCSC (none) -> C2941942; MANUFACTURER # GRM15XR71H561KA86J -> GCM155R71H561KA37D
- C39, C41, C42, C43: JLCPCB # C77020 -> (none); LCSC (none) -> C77020
- C40: JLCPCB # C77009 -> (none); LCSC (none) -> C77009
- C44: JLCPCB # C385032 -> (none); LCSC (none) -> C426094; MANUFACTURER # GRM155R61E225KE11D -> GRM155R61C475KE15D
- FB1: JLCPCB # C107335 -> (none); LCSC (none) -> C107335
- R40: JLCPCB # C137841 -> (none); LCSC (none) -> C137841
- R41: JLCPCB # C60490 -> (none); LCSC (none) -> C60490
- R42: JLCPCB # C106232 -> (none); LCSC (none) -> C106232
- TP7, TP8: now left out of the parts list
- U9: LCSC (none) -> C529358; MANUFACTURER (none) -> ST; MANUFACTURER # (none) -> STM32G431KBU6
Changed lines of the file:
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@@
-			)
-		)
-		(property "JLCPCB #" "C77020"
-			(at 166.37 142.24 0)
-			(effects
-				(font
-					(size 1.27 1.27)
-				)
-				(hide yes)
 			)
 		)
@@
 		)
 		(property "Manufacturer #" ""
+			(at 166.37 142.24 0)
+			(effects
+				(font
+					(size 1.27 1.27)
+				)
+				(hide yes)
+			)
+		)
+		(property "LCSC" "C77020"
 			(at 166.37 142.24 0)
 			(effects
@@
 			)
 		)
+		(property "LCSC" "C529358"
+			(at 147.32 133.35 0)
+			(effects
+				(font
+					(size 1.27 1.27)
+				)
+				(hide yes)
+			)
+		)
+		(property "MANUFACTURER" "ST"
+			(at 147.32 133.35 0)
+			(effects
+				(font
+					(size 1.27 1.27)
+				)
+				(hide yes)
+			)
+		)
+		(property "MANUFACTURER #" "STM32G431KBU6"
+			(at 147.32 133.35 0)
+			(effects
+				(font
+					(size 1.27 1.27)
+				)
+				(hide yes)
+			)
+		)
 		(pin "19"
 		)
@@
 			)
 		)
-		(property "JLCPCB #" "C385032"
-			(at 185.42 142.24 0)
-			(effects
-				(font
-					(size 1.27 1.27)
-				)
-				(hide yes)
-			)
-		)
 		(property "MANUFACTURER" "Murata"
 			(at 185.42 142.24 0)
@@
 			)
 		)
-		(property "MANUFACTURER #" "GRM155R61E225KE11D"
+		(property "MANUFACTURER #" "GRM155R61C475KE15D"
 			(at 185.42 142.24 0)
 			(effects
@@
 		)
 		(property "Manufacturer #" ""
+			(at 185.42 142.24 0)
+			(effects
+				(font
+					(size 1.27 1.27)
+				)
+				(hide yes)
+			)
+		)
+		(property "LCSC" "C426094"
 			(at 185.42 142.24 0)
 			(effects
@@
 			)
 		)
-		(property "JLCPCB #" "C77020"
-			(at 113.03 62.23 0)
-			(effects
-				(font
-					(size 1.27 1.27)
-				)
-				(hide yes)
-			)
-		)
 		(property "MANUFACTURER" "Murata"
 			(at 113.03 62.23 0)
@@
 		)
 		(property "Manufacturer #" ""
+			(at 113.03 62.23 0)
+			(effects
+				(font
+					(size 1.27 1.27)
+				)
+				(hide yes)
+			)
+		)
+		(property "LCSC" "C77020"
 			(at 113.03 62.23 0)
 			(effects
@@
 			)
 		)
+		(property "LCSC" "C529358"
+			(at 149.86 55.88 0)
+			(effects
+				(font
+					(size 1.27 1.27)
+				)
+				(hide yes)
+			)
+		)
+		(property "MANUFACTURER" "ST"
+			(at 149.86 55.88 0)
+			(effects
+				(font
+					(size 1.27 1.27)
+				)
+				(hide yes)
+			)
+		)
+		(property "MANUFACTURER #" "STM32G431KBU6"
+			(at 149.86 55.88 0)
+			(effects
+				(font
+					(size 1.27 1.27)
+				)
+				(hide yes)
+			)
+		)
 		(pin "19"
 			(alternate "USART1_TX")
@@
 			)
 		)
-		(property "JLCPCB #" "C60490"
-			(at 113.03 48.26 0)
-			(effects
-				(font
-					(size 1.27 1.27)
-				)
-				(hide yes)
-			)
-		)
 		(property "Package" "0402"
 			(at 115.824 48.514 0)
@@
 		)
 		(property "Manufacturer #" ""
+			(at 113.03 48.26 0)
+			(effects
+				(font
+					(size 1.27 1.27)
+				)
+				(hide yes)
+			)
+		)
+		(property "LCSC" "C60490"
 			(at 113.03 48.26 0)
 			(effects
@@
 		(unit 1)
 		(exclude_from_sim no)
-		(in_bom yes)
+		(in_bom no)
 		(on_board yes)
 		(dnp no)
@@
 			)
 		)
-		(property "JLCPCB #" "C137841"
-			(at 104.14 110.49 0)
-			(effects
-				(font
-					(size 1.27 1.27)
-				)
-				(hide yes)
-			)
-		)
 		(property "MANUFACTURER" "YAGEO"
 			(at 104.14 110.49 0)
@@
 		)
 		(property "MANUFACTURER #" "RC0402JR-0775RL"
+			(at 104.14 110.49 0)
+			(effects
+				(font
+					(size 1.27 1.27)
+				)
+				(hide yes)
+			)
+		)
+		(property "LCSC" "C137841"
 			(at 104.14 110.49 0)
 			(effects
@@
 			)
 		)
-		(property "JLCPCB #" "C106232"
-			(at 114.3 87.63 0)
-			(effects
-				(font
-					(size 1.27 1.27)
-				)
-				(hide yes)
-			)
-		)
 		(property "Package" "0402"
 			(at 114.3 87.63 90)
@@
 		(property "Manufacturer #" ""
 			(at 114.3 87.63 0)
+			(effects
+				(font
+					(size 1.27 1.27)
+				)
+				(hide yes)
+			)
+		)
+		(property "LCSC" "C106232"
+			(at 114.3 87.63 90)
 			(effects
 				(font
@@
 			)
 		)
-		(property "JLCPCB #" "C107335"
-			(at 104.14 135.89 90)
-			(effects
-				(font
-					(size 1.27 1.27)
-				)
-				(hide yes)
-			)
-		)
 		(property "MANUFACTURER" "TDK"
 			(at 104.14 135.89 90)
@@
 		)
 		(property "Package" "0603"
+			(at 104.14 135.89 90)
+			(effects
+				(font
+					(size 1.27 1.27)
+				)
+				(hide yes)
+			)
+		)
+		(property "LCSC" "C107335"
 			(at 104.14 135.89 90)
 			(effects
@@
 			)
 		)
-		(property "JLCPCB #" "C77020"
-			(at 128.27 140.97 0)
-			(effects
-				(font
-					(size 1.27 1.27)
-				)
-				(hide yes)
-			)
-		)
 		(property "MANUFACTURER" "Murata"
 			(at 128.27 140.97 0)
@@
 		)
 		(property "Manufacturer #" ""
+			(at 128.27 140.97 0)
+			(effects
+				(font
+					(size 1.27 1.27)
+				)
+				(hide yes)
+			)
+		)
+		(property "LCSC" "C77020"
 			(at 128.27 140.97 0)
 			(effects
@@
 			)
 		)
-		(property "JLCPCB #" "C77009 "
-			(at 116.84 140.97 0)
-			(effects
-				(font
-					(size 1.27 1.27)
-				)
-				(hide yes)
-			)
-		)
 		(property "MANUFACTURER" "Murata"
 			(at 116.84 140.97 0)
@@
 		)
 		(property "Manufacturer #" ""
+			(at 116.84 140.97 0)
+			(effects
+				(font
+					(size 1.27 1.27)
+				)
+				(hide yes)
+			)
+		)
+		(property "LCSC" "C77009 "
 			(at 116.84 140.97 0)
 			(effects
@@
 			)
 		)
-		(property "JLCPCB #" "C21012317"
-			(at 104.14 91.44 0)
-			(effects
-				(font
-					(size 1.27 1.27)
-				)
-				(hide yes)
-			)
-		)
 		(property "MANUFACTURER" "Murata"
 			(at 104.14 91.44 0)
@@
 			)
 		)
-		(property "MANUFACTURER #" "GRM15XR71H561KA86J"
+		(property "MANUFACTURER #" "GCM155R71H561KA37D"
 			(at 104.14 91.44 0)
 			(effects
@@
 		)
 		(property "Manufacturer #" ""
+			(at 104.14 91.44 0)
+			(effects
+				(font
+					(size 1.27 1.27)
+				)
+				(hide yes)
+			)
+		)
+		(property "LCSC" "C2941942"
 			(at 104.14 91.44 0)
 			(effects
@@
 		(unit 1)
 		(exclude_from_sim no)
-		(in_bom yes)
+		(in_bom no)
 		(on_board yes)
 		(dnp no)
@@
 			)
 		)
-		(property "JLCPCB #" "C77020"
-			(at 175.26 142.24 0)
-			(effects
-				(font
-					(size 1.27 1.27)
-				)
-				(hide yes)
-			)
-		)
 		(property "MANUFACTURER" "Murata"
 			(at 175.26 142.24 0)
@@
 			(at 175.26 142.24 0)
 			(effects
+				(font
+					(size 1.27 1.27)
+				)
+				(hide yes)
+			)
+		)
+		(property "LCSC" "C77020"
+			(at 175.26 142.24 0)
+			(effects
