File: polski_fc.kicad_pcb (KiCad board)
At the start: 8 copper layers, 37 x 37 mm, 157 parts, among them J2 JST-SH 1x08, J3 Digital_VTX_Connector, J4 UJ20-C-H-G-SMT-5-P16-TR, P1 4V5, P10 R1, P11 +, P12 C, P13 R5, P14 M1, P15 M2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

Commit message: Updated
Routing:
- net GND: vias 152 -> 153
Other:
- board text added: "v0.1"
